File: daplink-hdk/daplink-hdk.kicad_sch (KiCad schematic)
At the start: 48 parts, among them J3 Conn_01x12_Socket, J3 Conn_02x05_Odd_Even, J3 USB_C_Receptacle_USB2.0, J4 Conn_02x05_Odd_Even, J5 Conn_01x12_Socket, J6 Conn_01x03, Q1 DMP3099L, Q3 DMN3023L-7, SW1 SW_Push, U1 ESDS302DBVR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

Commit message: Fix missing power LED trace, increment rev, and add Gitlab CI
Parts:
- U1: MFP (none) -> ESDS302DBVR
Changed lines of the file:
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@@
     (title "daplink-hdk")
     (date "2023-10-27")
-    (rev "Rev A")
+    (rev "Rev B")
     (company "everyday dev")
     (comment 1 "License: CC-BY-SA")
@@
       (effects (font (size 1.27 1.27)) hide)
     )
+    (property "MFP" "ESDS302DBVR" (at 58.42 48.26 0)
+      (effects (font (size 1.27 1.27)) hide)
+    )
